Commit message: update urdf

File: share/model/DoubleArmV7/original/urdf/DoubleArmV7A.urdf (robot description, URDF)
Before this commit: robot DoubleArmV7-Upper, 46 links, 45 joints
Links:
- link HANDLNK_I: geometry collision box size=0.02 0.028 0.01; collision box size=0.02 0.028 0.01
- link HANDLNK_O: geometry collision box size=0.02 0.028 0.01; collision box size=0.02 0.028 0.01
- link HANDSLNK_I: geometry collision box size=0.08 0.028 0.028; collision cylinder length=0.028 radius=0.014
- link HANDSLNK_O: geometry collision box size=0.08 0.028 0.042; collision cylinder length=0.042 radius=0.014
- link HANDTIP_L: geometry collision box size=0.004 0.012 0.00314; collision box size=0.004 0.012 0.00314
- link HANDTIP_U: geometry collision box size=0.004 0.012 0.00314; collision box size=0.004 0.012 0.00314
- link MANIARM: geometry visual mesh filename=DoubleArmV7-Upper-MANIARM-visual-0.dae scale=1.0000000000000013 1.000000000000002 1.0000000000000016
- link MANIFNG_L: geometry collision box size=0.01 0.048364 0.014; collision box size=0.016 0.02 0.01
- link MANIFNG_U: geometry collision box size=0.01 0.048364 0.014; collision box size=0.016 0.02 0.01
Joints:
- joint ARM: origin xyz=-1.7599999999999996 1.3322676295501878e-15 1.1102230246251565e-16 rpy=0.0 -0.0 0.0 -> xyz=-1.7599999999999993 5.551115123125783e-16 -9.71445146547012e-17 rpy=0.0 -0.0 0.0
- joint BLOCK: origin xyz=0.845 -0.11 0.19199999999999995 rpy=0.0 -0.0 0.0 -> xyz=0.845 -0.11 0.192 rpy=0.0 -0.0 0.0
- joint BOOM: origin xyz=0.06999999999999984 -3.608224830031759e-16 0.20000000000000007 rpy=1.57079632679 8.65956056235e-17 3.14159265359 -> xyz=0.0700000000000004 1.5265566588595902e-16 0.20000000000000012 rpy=1.57079632679 8.65956056235e-17 3.14159265359
- joint HANDBASE: origin xyz=0.0 1.0547118733938987e-15 -0.4053000000000009 rpy=0.0 -0.0 0.0 -> xyz=-4.440892098500626e-16 -2.7755575615628914e-17 -0.40529999999999977 rpy=0.0 -0.0 0.0
- joint HANDLNK_I: origin xyz=1.1102230246251565e-16 0.006500000000000783 -0.15500000000000025 rpy=1.57079632679 1.45266895236 1.78987944049e-14 -> xyz=-1.1102230246251565e-16 0.006499999999999978 -0.15499999999999992 rpy=1.57079632679 1.45266895236 4.23918814852e-15
- joint HANDLNK_O: origin xyz=1.1102230246251565e-16 -0.006499999999999201 -0.15500000000000025 rpy=1.57079632679 1.45266922743 3.14159265359 -> xyz=-1.1102230246251565e-16 -0.0065000000000000335 -0.15499999999999992 rpy=1.57079632679 1.45266922743 3.14159265359
- joint HANDSLNK_I: origin xyz=-1.1102230246251565e-16 3.608224830031759e-16 4.440892098500626e-16 rpy=-1.57079632679 0.502146933762 3.14159265359 -> xyz=1.1102230246251565e-16 3.885780586188048e-16 1.1102230246251565e-16 rpy=-1.57079632679 0.502146933762 3.14159265359
- joint HANDSLNK_O: origin xyz=-1.1102230246251565e-16 3.608224830031759e-16 4.440892098500626e-16 rpy=1.57079632679 0.502146933762 -3.16645213446e-17 -> xyz=1.1102230246251565e-16 3.885780586188048e-16 1.1102230246251565e-16 rpy=1.57079632679 0.502146933762 1.89987128067e-16
- joint HANDTIP_L: origin xyz=0.17100000000000004 0.0 -1.942890293094024e-16 rpy=-2.80434529179e-16 1.00458830582e-16 -0.118127374433 -> xyz=0.17099999999999982 4.440892098500626e-16 3.0531133177191805e-16 rpy=-9.18211105227e-19 9.17549819597e-17 -0.118127374433
- joint HANDTIP_U: origin xyz=0.17100000000000015 -4.440892098500626e-16 0.0 rpy=1.68550260069e-17 -6.51459040917e-17 -0.118127374433 -> xyz=0.1710000000000006 -2.220446049250313e-16 -3.885780586188048e-16 rpy=-3.54187949632e-16 -1.17224040023e-16 -0.118127374433
- joint MANIARM: origin xyz=-1.48 0.08000000000000063 -4.163336342344337e-16 rpy=0.0 -0.0 3.14159265359 -> xyz=-1.4799999999999995 0.0800000000000003 -4.718447854656915e-16 rpy=0.0 -0.0 3.14159265359
- joint MANIBOOM: origin xyz=0.06999999999999973 -3.608224830031759e-16 0.14000000000000035 rpy=-1.57079632679 1.57079632679 0.0 -> xyz=0.07000000000000028 1.942890293094024e-16 0.1400000000000003 rpy=-1.57079632679 1.57079632679 0.0
- joint MANIELBOW: origin xyz=-0.5499999999999989 0.2700000000000006 4.718447854656915e-16 rpy=1.57079632679 7.77156117238e-16 1.57079632679 -> xyz=-0.5499999999999989 0.27000000000000035 1.942890293094024e-16 rpy=1.57079632679 1.16573417586e-15 1.57079632679
- joint MANIFNG_L: origin xyz=-0.029999999999999805 8.049116928532385e-16 -0.14000000000000035 rpy=1.57079632679 1.45266922743 3.14159265359 -> xyz=-0.030000000000000027 0.0 -0.1399999999999999 rpy=1.57079632679 1.45266922743 3.14159265359
- joint MANIFNG_U: origin xyz=0.030000000000000138 7.771561172376096e-16 -0.14000000000000035 rpy=1.57079632679 1.45266895236 1.78987944049e-14 -> xyz=0.029999999999999916 -2.7755575615628914e-17 -0.1399999999999999 rpy=1.57079632679 1.45266895236 4.23918814852e-15
- joint MFRAME: origin xyz=0.0 0.0 0.52 rpy=0.0 -0.0 0.0 -> xyz=0.0 0.0 0.0 rpy=0.0 -0.0 0.0
- joint MNP_SWING: origin xyz=0.5595 -0.13 0.118 rpy=0.0 -0.0 0.0 -> xyz=0.5595 -0.13 0.11800000000000005 rpy=0.0 -0.0 0.0
- joint PUSHROD: origin xyz=2.220446049250313e-16 7.771561172376096e-16 -0.09170000000000034 rpy=0.0 -0.0 0.0 -> xyz=-1.1102230246251565e-16 -2.7755575615628914e-17 -0.0917 rpy=0.0 -0.0 0.0
- joint TOHKU_PITCH: origin xyz=-0.9649999999999999 -1.1102230246251565e-16 2.914335439641036e-16 rpy=1.57079632679 1.16573417586e-15 1.57079632679 -> xyz=-0.9649999999999999 1.6653345369377348e-16 -5.551115123125783e-17 rpy=1.57079632679 -1.11022302463e-16 1.57079632679
- joint TOHKU_ROLL: origin xyz=4.440892098500626e-16 1.5543122344752192e-15 -0.22699999999999942 rpy=0.0 -0.0 0.0 -> xyz=9.992007221626409e-16 1.3183898417423734e-15 -0.22699999999999942 rpy=0.0 -0.0 0.0
- joint TOHKU_TIP_01: origin xyz=-1.1102230246251565e-16 1.942890293094024e-16 -0.3089999999999997 rpy=0.0 -0.0 0.0 -> xyz=9.992007221626409e-16 -7.077671781985373e-16 -0.3089999999999997 rpy=0.0 -0.0 0.0
- joint TOHKU_TIP_02: origin xyz=-1.1102230246251565e-16 1.942890293094024e-16 -0.3089999999999997 rpy=0.0 -0.0 3.14159265359 -> xyz=9.992007221626409e-16 -7.077671781985373e-16 -0.3089999999999997 rpy=0.0 -0.0 3.14159265359
- joint UFRAME: origin xyz=0.0 0.0 0.8200000000000001 rpy=0.0 -0.0 3.14159265359 -> xyz=0.0 0.0 0.3 rpy=0.0 -0.0 3.14159265359
- joint WHEEL_L0: origin xyz=0.74 0.6 0.22500000000000003 rpy=0.0 -0.0 0.0 -> xyz=0.74 0.6 -0.295 rpy=0.0 -0.0 0.0
- joint WHEEL_L1: origin xyz=0.26 0.6 0.22500000000000003 rpy=0.0 -0.0 0.0 -> xyz=0.26 0.6 -0.295 rpy=0.0 -0.0 0.0
- joint WHEEL_L2: origin xyz=-0.22 0.6 0.22500000000000003 rpy=0.0 -0.0 0.0 -> xyz=-0.22 0.6 -0.295 rpy=0.0 -0.0 0.0
- joint WHEEL_L3: origin xyz=-0.7 0.6 0.22500000000000003 rpy=0.0 -0.0 0.0 -> xyz=-0.7 0.6 -0.295 rpy=0.0 -0.0 0.0
- joint WHEEL_R0: origin xyz=0.74 -0.6 0.22500000000000003 rpy=0.0 -0.0 0.0 -> xyz=0.74 -0.6 -0.295 rpy=0.0 -0.0 0.0
- joint WHEEL_R1: origin xyz=0.26 -0.6 0.22500000000000003 rpy=0.0 -0.0 0.0 -> xyz=0.26 -0.6 -0.295 rpy=0.0 -0.0 0.0
- joint WHEEL_R2: origin xyz=-0.22 -0.6 0.22500000000000003 rpy=0.0 -0.0 0.0 -> xyz=-0.22 -0.6 -0.295 rpy=0.0 -0.0 0.0
- joint WHEEL_R3: origin xyz=-0.7 -0.6 0.22500000000000003 rpy=0.0 -0.0 0.0 -> xyz=-0.7 -0.6 -0.295 rpy=0.0 -0.0 0.0
- joint WIRE_GUARD_L: origin xyz=0.02 0.61 0.2 rpy=0.0 -0.0 0.0 -> xyz=0.02 0.61 -0.32 rpy=0.0 -0.0 0.0
- joint WIRE_GUARD_R: origin xyz=0.02 -0.61 0.2 rpy=0.0 -0.0 0.0 -> xyz=0.02 -0.61 -0.32 rpy=0.0 -0.0 0.0
- joint YAWJOINT: origin xyz=-3.3306690738754696e-16 3.608224830031759e-16 -0.23000000000000043 rpy=0.0 -0.0 0.0 -> xyz=-4.440892098500626e-16 5.273559366969494e-16 -0.2300000000000002 rpy=0.0 -0.0 0.0
